File: ESP32.kicad_sch (KiCad schematic)
At the start: 8 parts, among them J9 PROG, SW2 RESET, SW3 BOOT, U2 ESP32-WROOM-32D

Commit message: Started to change project in preparation for next version
Parts:
- renumbered J9 to J8, R6 to R5, SW2 to SW1, SW3 to SW2

Commit message: Submitted V0.2 to production
Parts:
- removed C3: 10u, Capacitor_SMD:C_1206_3216Metric, symbol Device:C
- added R6: 10k, Resistor_SMD:R_0603_1608Metric_Pad0.98x0.95mm_HandSolder, symbol Device:R
- SW1: value RESET -> Reset; footprint Button_Switch_SMD:SW_Push_1P1T_NO_CK_KSC7xxJ -> Button_Switch_SMD:SW_Push_1P1T_XKB_TS-1187A; LCSC C318884 -> (none)
- SW2: value BOOT -> Boot; footprint Button_Switch_SMD:SW_Push_1P1T_NO_CK_KSC7xxJ -> Button_Switch_SMD:SW_Push_1P1T_XKB_TS-1187A; LCSC C318884 -> (none)
- U3: renamed from U2; footprint RF_Module:ESP32-WROOM-32 -> RF_Module:ESP32-WROOM-32D
- renumbered J8 to J7
Connections:
- net +3V3: now also R6.2
- net BOOT: now also R6.1
- net BUTTON renamed INT2
- net NPX2 renamed INT1
Other:
- moved on the sheet: C4
